File: hw/RemBreak/power_control.kicad_sch (KiCad schematic)
At the start: 24 parts, among them Q10 BC337, Q11 BC847, Q12 Si7141DP, Q13 BC337, Q14 BC847, U6 BD4830FVE-TR

Commit message: temporary schematics sheets
Parts:
- added C1: 0.1uF, symbol Device:C_Polarized
- added C5: 100nF, symbol Device:C
- added IC1: LTC2943IDD#TRPBF, SON50P300X300X80-9N-D, symbol dodo-device:LTC2943IDD#TRPBF
- added IC2: MAX17049G+T10, Package_DFN_QFN:TDFN-8-1EP_2x2mm_P0.5mm_EP0.8x1.2mm, symbol dodo-power:MAX17049G+T10
- added R16, R18: 10, symbol Device:R
- added R19, R23: 10k, symbol Device:R
- added U2: INA219BxDCN, Package_TO_SOT_SMD:SOT-23-8, symbol Analog_ADC:INA219BxDCN
Connections:
- net +BATT: now also C1.1, IC2.2 (CELL)
- net GND: now also C1.2, IC2.1 (CTG), IC2.4 (GND_1), IC2.6 (QSTRT), IC2.9 (GND_2), U2.3 (GND), U2.7 (A0), U2.8 (A1)
- net BAT+ renamed CS_IN+
- net CONNECTED: no longer names the net of Q11.1 (B), R2.2, R32.2, R33.1, R4.2
- net SW+: no longer names the net of Q12.4 (G), R35.2
- net SW-: no longer names the net of Q13.1 (C), Q14.3 (C)
- net VOUT: no longer names the net of Q12.5 (D)
- new net: C5.1, R18.2, U2.2 (IN-)
- new net: C5.2, R16.2, U2.1 (IN+)
- new net +3V3: IC2.3 (VDD), R19.1, R23.1, U2.4 (VS)
- new net BATT_ALRM: IC2.5 (~{ALRT})
- new net IN+: R16.1
- new net IN-: R18.1
- new net SCL: IC2.7 (SCL), R19.2, U2.5 (SCL)
- new net SDA: IC2.8 (SDA), R23.2, U2.6 (SDA)
Other:
- note added: "BATTERY SoC IC I2C address: 0x36 + R/W"
- note added: "CURRENT SENSOR I2C address: 0x40 + R/W"
- moved on the sheet: C4, D4, Q10, Q11, Q12, Q13, Q14, R1, R2, R28, R29, R30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
