File: hw/RemBreak/power_switch.kicad_sch (KiCad schematic)
At the start: 41 parts, among them J12 Conn_01x01, J14 Conn_01x01, Q11 BC337, Q12 BC847, Q3 BC847, Q6 BC337, Q7 BC847, Q8 SiS415DNT, Q9 BC337, U1 L7805, U2 L7805, U3 XC6220B331MR, U4 MAX40200AUK, U8 BD48ExxG, U9 BD48ExxG

Commit message: schematics development in progress
Connections:
- net PWR: no longer C1.1, Q8.1 (S), Q8.2 (S), Q8.3 (S), U1.1 (IN), U2.1 (IN)
- net VBATT: now also Q8.1 (S), Q8.2 (S), Q8.3 (S); no longer Q8.5 (D)
- net EN: now reaches R30.1, R34.1, R35.1, R43.1, R44.1, U9.1 (VOUT)
- new net 7V4: C1.1, Q8.5 (D), U1.1 (IN), U2.1 (IN)
Other:
- moved on the sheet: Q8, R23, R42
Changed lines of the file:
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@@
 	)
 	(junction
-		(at 217.17 127)
+		(at 217.17 124.46)
 		(diameter 0)
 		(color 0 0 0 0)
@@
 	)
 	(junction
+		(at 184.15 140.97)
+		(diameter 0)
+		(color 0 0 0 0)
+	)
+	(junction
 		(at 199.39 59.69)
 		(diameter 0)
@@
 		(color 0 0 0 0)
 	)
+	(bus_entry
+		(at 269.24 59.69)
+		(size 2.54 2.54)
+		(stroke
+			(width 0)
+			(type default)
+		)
+	)
+	(bus_entry
+		(at 269.24 38.1)
+		(size 2.54 2.54)
+		(stroke
+			(width 0)
+			(type default)
+		)
+	)
+	(bus_entry
+		(at 269.24 49.53)
+		(size 2.54 2.54)
+		(stroke
+			(width 0)
+			(type default)
+		)
+	)
 	(wire
 		(pts
@@
 		)
 	)
+	(bus
+		(pts
+			(xy 271.78 72.39) (xy 273.05 72.39)
+		)
+		(stroke
+			(width 0)
+			(type default)
+		)
+	)
 	(wire
 		(pts
@@
 	(wire
 		(pts
-			(xy 266.7 59.69) (xy 271.78 59.69)
+			(xy 266.7 59.69) (xy 269.24 59.69)
 		)
 		(stroke
@@
 	(wire
 		(pts
-			(xy 217.17 110.49) (xy 217.17 127)
+			(xy 217.17 110.49) (xy 217.17 124.46)
 		)
 		(stroke
@@
 	(wire
 		(pts
-			(xy 184.15 88.9) (xy 271.78 88.9)
+			(xy 184.15 88.9) (xy 273.05 88.9)
 		)
 		(stroke
@@
 	(wire
 		(pts
-			(xy 199.39 49.53) (xy 271.78 49.53)
+			(xy 199.39 49.53) (xy 269.24 49.53)
 		)
 		(stroke
@@
 	(wire
 		(pts
-			(xy 29.21 96.52) (xy 29.21 105.41)
+			(xy 29.21 92.71) (xy 29.21 105.41)
 		)
 		(stroke
@@
 	(wire
 		(pts
-			(xy 29.21 68.58) (xy 29.21 88.9)
+			(xy 29.21 68.58) (xy 29.21 85.09)
 		)
 		(stroke
@@
 	(wire
 		(pts
-			(xy 234.95 121.92) (xy 234.95 135.89)
+			(xy 234.95 121.92) (xy 234.95 133.35)
 		)
 		(stroke
@@
 	(wire
 		(pts
-			(xy 156.21 38.1) (xy 271.78 38.1)
+			(xy 156.21 38.1) (xy 269.24 38.1)
+		)
+		(stroke
+			(width 0)
+			(type default)
+		)
+	)
+	(bus
+		(pts
+			(xy 271.78 52.07) (xy 271.78 62.23)
 		)
 		(stroke
@@
 		)
 	)
+	(bus
+		(pts
+			(xy 271.78 62.23) (xy 271.78 72.39)
+		)
+		(stroke
+			(width 0)
+			(type default)
+		)
+	)
 	(wire
 		(pts
@@
 	(wire
 		(pts
+			(xy 184.15 140.97) (xy 273.05 140.97)
+		)
+		(stroke
+			(width 0)
+			(type default)
+		)
+	)
+	(wire
+		(pts
 			(xy 82.55 121.92) (xy 82.55 127)
 		)
@@
 	(wire
 		(pts
-			(xy 217.17 127) (xy 217.17 128.27)
+			(xy 217.17 124.46) (xy 217.17 125.73)
 		)
 		(stroke
@@
 	(wire
 		(pts
-			(xy 199.39 127) (xy 217.17 127)
+			(xy 199.39 124.46) (xy 217.17 124.46)
 		)
 		(stroke
@@
 	(wire
 		(pts
-			(xy 199.39 127) (xy 199.39 110.49)
+			(xy 199.39 124.46) (xy 199.39 110.49)
 		)
 		(stroke
@@
 		)
 	)
+	(bus
+		(pts
+			(xy 271.78 40.64) (xy 271.78 52.07)
+		)
+		(stroke
+			(width 0)
+			(type default)
+		)
+	)
+	(bus
+		(pts
+			(xy 271.78 29.21) (xy 271.78 40.64)
+		)
+		(stroke
+			(width 0)
+			(type default)
+		)
+	)
 	(wire
 		(pts
@@
 		)
 	)
-	(hierarchical_label "5V"
-		(shape output)
-		(at 271.78 49.53 0)
+	(label "3V3"
+		(at 266.7 59.69 0)
 		(fields_autoplaced yes)
 		(effects
@@
 				(size 1.27 1.27)
 			)
-			(justify left)
+			(justify left bottom)
+		)
+	)
+	(label "5V"
+		(at 266.7 49.53 0)
+		(fields_autoplaced yes)
+		(effects
+			(font
+				(size 1.27 1.27)
+			)
+			(justify left bottom)
+		)
+	)
+	(label "7V4"
+		(at 266.7 38.1 0)
+		(fields_autoplaced yes)
+		(effects
+			(font
+				(size 1.27 1.27)
+			)
+			(justify left bottom)
 		)
 	)
-	(hierarchical_label "3V3"
+	(hierarchical_label "EN"
 		(shape output)
-		(at 271.78 59.69 0)
+		(at 273.05 140.97 0)
 		(fields_autoplaced yes)
 		(effects
@@
 	(hierarchical_label "PWR"
 		(shape output)
-		(at 271.78 38.1 0)
+		(at 273.05 72.39 0)
 		(fields_autoplaced yes)
 		(effects
@@
 	(hierarchical_label "VBUS"
 		(shape input)
-		(at 271.78 88.9 0)
+		(at 273.05 88.9 0)
 		(fields_autoplaced yes)
 		(effects
@@
 	(symbol
 		(lib_id "Device:R")
-		(at 29.21 92.71 180)
+		(at 29.21 88.9 180)
 		(unit 1)
 		(exclude_from_sim no)
@@
 		(dnp no)
 		(property "Reference" "R23"
-			(at 26.924 92.71 90)
+			(at 26.924 88.9 90)
 			(effects
 				(font
@@
 		)
 		(property "Value" "50k"
-			(at 32.004 92.71 90)
+			(at 32.004 88.9 90)
 			(effects
 				(font
@@
 		)
 		(property "Footprint" "Resistor_SMD:R_0805_2012Metric"
-			(at 30.988 92.71 90)
+			(at 30.988 88.9 90)
 			(effects
 				(font
@@
 		)
 		(property "Datasheet" "~"
-			(at 29.21 92.71 0)
+			(at 29.21 88.9 0)
 			(effects
 				(font
@@
 		)
 		(property "Description" "Resistor"
-			(at 29.21 92.71 0)
+			(at 29.21 88.9 0)
 			(effects
 				(font
@@
 	(symbol
 		(lib_id "Device:R")
-		(at 217.17 132.08 180)
+		(at 217.17 129.54 180)
 		(unit 1)
 		(exclude_from_sim no)
@@
 		(fields_autoplaced yes)
 		(property "Reference" "R42"
-			(at 219.71 130.8099 0)
+			(at 219.71 128.2699 0)
 			(effects
 				(font
@@
 		)
 		(property "Value" "4k2"
-			(at 219.71 133.3499 0)
+			(at 219.71 130.8099 0)
 			(effects
 				(font
@@
 		)
 		(property "Footprint" "Resistor_SMD:R_0805_2012Metric"
-			(at 218.948 132.08 90)
+			(at 218.948 129.54 90)
 			(effects
 				(font
@@
 		)
 		(property "Datasheet" "~"
-			(at 217.17 132.08 0)
+			(at 217.17 129.54 0)
 			(effects
 				(font
@@
 		)
 		(property "Description" "Resistor"
-			(at 217.17 132.08 0)
+			(at 217.17 129.54 0)
 			(effects
 				(font
@@
 	(symbol
 		(lib_id "Transistor_FET:SiS415DNT")
-		(at 109.22 40.64 90)
+		(at 109.22 40.64 270)
+		(mirror x)
 		(unit 1)
 		(exclude_from_sim no)
@@
 		(on_board yes)
 		(dnp no)
-		(fields_autoplaced yes)
 		(property "Reference" "Q8"
 			(at 109.22 33.02 90)
@@
 		)
 		(property "Footprint" "Package_SO:Vishay_PowerPAK_1212-8_Single"
-			(at 111.125 35.56 0)
+			(at 107.315 35.56 0)
 			(effects
 				(font
@@
 		)
 		(property "Datasheet" "https://www.vishay.com/docs/63684/sis415dnt.pdf"
-			(at 113.03 35.56 0)
+			(at 105.41 35.56 0)
 			(effects
 				(font
@@
 	(symbol
 		(lib_id "power:GND")
-		(at 234.95 135.89 0)
+		(at 234.95 133.35 0)
 		(unit 1)
 		(exclude_from_sim no)
@@
 		(dnp no)
 		(property "Reference" "#PWR010"
-			(at 234.95 142.24 0)
+			(at 234.95 139.7 0)
 			(effects
 				(font
@@
 		)
 		(property "Value" "GND"
-			(at 234.95 140.97 0)
+			(at 234.95 138.43 0)
 			(effects
 				(font
@@
 		)
 		(property "Footprint" ""
-			(at 234.95 135.89 0)
+			(at 234.95 133.35 0)
 			(effects
 				(font
@@
 		)
 		(property "Datasheet" ""
-			(at 234.95 135.89 0)
+			(at 234.95 133.35 0)
 			(effects
 				(font
@@
 		)
 		(property "Description" "Power symbol creates a global label with name \"GND\" , ground"
-			(at 234.95 135.89 0)
+			(at 234.95 133.35 0)
 			(effects
 				(font
@@
 	(symbol
 		(lib_id "power:GND")
-		(at 217.17 135.89 0)
+		(at 217.17 133.35 0)
 		(unit 1)
 		(exclude_from_sim no)
@@
 		(dnp no)
 		(property "Reference" "#PWR016"
-			(at 217.17 142.24 0)
+			(at 217.17 139.7 0)
 			(effects
 				(font
@@
 		)
 		(property "Value" "GND"
-			(at 217.17 140.97 0)
+			(at 217.17 138.43 0)
 			(effects
 				(font
@@
 		)
 		(property "Footprint" ""
-			(at 217.17 135.89 0)
+			(at 217.17 133.35 0)
 			(effects
 				(font
@@
 		)
 		(property "Datasheet" ""
-			(at 217.17 135.89 0)
+			(at 217.17 133.35 0)
 			(effects
 				(font
@@
 		)
 		(property "Description" "Power symbol creates a global label with name \"GND\" , ground"
-			(at 217.17 135.89 0)
+			(at 217.17 133.35 0)
 			(effects
 				(font

Commit message: updated pcb and schematics - still in progress
Parts:
- removed J12, J14: Conn_01x01, TestPoint:TestPoint_Pad_2.5x2.5mm, symbol Connector_Generic:Conn_01x01
- U2: footprint Package_TO_SOT_THT:TO-220-3_Horizontal_TabDown -> Package_TO_SOT_THT:TO-220-3_Vertical
Connections:
- net 7V4: no longer C1.1, U1.1 (IN), U2.1 (IN)
- net SW-: now reaches R23.2, R25.2
- net SW-: now also C1.1, U1.1 (IN), U2.1 (IN)
- net VBATT renamed SW+
Changed lines of the file:
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@@
 	)
 	(junction
-		(at 82.55 68.58)
-		(diameter 0)
-		(color 0 0 0 0)
-	)
-	(junction
 		(at 109.22 49.53)
 		(diameter 0)
@@
 	)
 	(junction
-		(at 156.21 38.1)
-		(diameter 0)
-		(color 0 0 0 0)
-	)
-	(junction
 		(at 185.42 49.53)
 		(diameter 0)
@@
 	)
 	(junction
+		(at 156.21 49.53)
+		(diameter 0)
+		(color 0 0 0 0)
+	)
+	(junction
 		(at 207.01 76.2)
 		(diameter 0)
@@
 	)
 	(junction
-		(at 29.21 105.41)
+		(at 82.55 64.77)
 		(diameter 0)
 		(color 0 0 0 0)
 	)
 	(junction
-		(at 156.21 49.53)
+		(at 29.21 105.41)
 		(diameter 0)
 		(color 0 0 0 0)
@@
 	(wire
 		(pts
-			(xy 156.21 38.1) (xy 156.21 49.53)
-		)
-		(stroke
-			(width 0)
-			(type default)
-		)
-	)
-	(wire
-		(pts
 			(xy 266.7 59.69) (xy 269.24 59.69)
 		)
@@
 	(wire
 		(pts
+			(xy 135.89 49.53) (xy 156.21 49.53)
+		)
+		(stroke
+			(width 0)
+			(type default)
+		)
+	)
+	(wire
+		(pts
 			(xy 144.78 86.36) (xy 144.78 100.33)
 		)
@@
 	(wire
 		(pts
+			(xy 135.89 64.77) (xy 135.89 49.53)
+		)
+		(stroke
+			(width 0)
+			(type default)
+		)
+	)
+	(wire
+		(pts
 			(xy 29.21 92.71) (xy 29.21 105.41)
 		)
@@
 	(wire
 		(pts
-			(xy 29.21 68.58) (xy 29.21 85.09)
+			(xy 29.21 64.77) (xy 29.21 85.09)
 		)
 		(stroke
@@
 	(wire
 		(pts
-			(xy 82.55 68.58) (xy 82.55 71.12)
+			(xy 82.55 64.77) (xy 82.55 71.12)
 		)
 		(stroke
@@
 		)
 	)
-	(wire
+	(bus
 		(pts
-			(xy 156.21 38.1) (xy 269.24 38.1)
+			(xy 271.78 52.07) (xy 271.78 62.23)
 		)
 		(stroke
@@
 		)
 	)
-	(bus
+	(wire
 		(pts
-			(xy 271.78 52.07) (xy 271.78 62.23)
+			(xy 195.58 121.92) (xy 207.01 121.92)
 		)
 		(stroke
@@
 	(wire
 		(pts
-			(xy 195.58 121.92) (xy 207.01 121.92)
+			(xy 82.55 64.77) (xy 135.89 64.77)
 		)
 		(stroke
@@
 	(wire
 		(pts
+			(xy 26.67 55.88) (xy 82.55 55.88)
+		)
+		(stroke
+			(width 0)
+			(type default)
+		)
+	)
+	(wire
+		(pts
 			(xy 82.55 121.92) (xy 82.55 127)
 		)
@@
 	(wire
 		(pts
-			(xy 114.3 38.1) (xy 156.21 38.1)
+			(xy 114.3 38.1) (xy 269.24 38.1)
 		)
 		(stroke
@@
 	(wire
 		(pts
+			(xy 82.55 60.96) (xy 26.67 60.96)
+		)
+		(stroke
+			(width 0)
+			(type default)
+		)
+	)
+	(wire
+		(pts
 			(xy 156.21 62.23) (xy 156.21 60.96)
 		)
@@
 	(wire
 		(pts
-			(xy 82.55 68.58) (xy 29.21 68.58)
+			(xy 82.55 64.77) (xy 29.21 64.77)
 		)
 		(stroke
@@
 	(wire
 		(pts
-			(xy 82.55 60.96) (xy 82.55 68.58)
+			(xy 82.55 60.96) (xy 82.55 64.77)
 		)
 		(stroke
@@
 		)
 	)
+	(hierarchical_label "SW-"
+		(shape input)
+		(at 26.67 60.96 180)
+		(fields_autoplaced yes)
+		(effects
+			(font
+				(size 1.27 1.27)
+			)
+			(justify right)
+		)
+	)
+	(hierarchical_label "SW+"
+		(shape input)
+		(at 26.67 55.88 180)
+		(fields_autoplaced yes)
+		(effects
+			(font
+				(size 1.27 1.27)
+			)
+			(justify right)
+		)
+	)
 	(hierarchical_label "VBATT"
 		(shape input)
@@
 	)
 	(symbol
-		(lib_id "Connector_Generic:Conn_01x01")
-		(at 77.47 60.96 180)
-		(unit 1)
-		(exclude_from_sim no)
-		(in_bom yes)
-		(on_board yes)
-		(dnp no)
-		(property "Reference" "J12"
-			(at 75.184 60.96 0)
-			(effects
-				(font
-					(size 1.27 1.27)
-				)
-				(justify left)
-			)
-		)
-		(property "Value" "Conn_01x01"
-			(at 74.93 59.6901 0)
-			(effects
-				(font
-					(size 1.27 1.27)
-				)
-				(justify left)
-				(hide yes)
-			)
-		)
-		(property "Footprint" "TestPoint:TestPoint_Pad_2.5x2.5mm"
-			(at 77.47 60.96 0)
-			(effects
-				(font
-					(size 1.27 1.27)
-				)
-				(hide yes)
-			)
-		)
-		(property "Datasheet" "~"
-			(at 77.47 60.96 0)
-			(effects
-				(font
-					(size 1.27 1.27)
-				)
-				(hide yes)
-			)
-		)
-		(property "Description" "Generic connector, single row, 01x01, script generated (kicad-library-utils/schlib/autogen/connector/)"
-			(at 77.47 60.96 0)
-			(effects
-				(font
-					(size 1.27 1.27)
-				)
-				(hide yes)
-			)
-		)
-		(pin "1"
-		)
-		(instances
-			(project "RemBreak"
-				(path "/e6d4ae5b-c9d7-4cbe-b288-c929fdf55a75/2d0cc746-3115-4ebf-adba-86e7fd6ac8bd"
-					(reference "J12")
-					(unit 1)
-				)
-			)
-		)
-	)
-	(symbol
 		(lib_id "Device:R")
 		(at 82.55 130.81 0)
@@
 			)
 		)
-		(property "Footprint" "Package_TO_SOT_THT:TO-220-3_Horizontal_TabDown"
+		(property "Footprint" "Package_TO_SOT_THT:TO-220-3_Vertical"
 			(at 172.085 67.31 0)
 			(effects
@@
 					(unit 1)
 				)
-			)
-		)
-	)
-	(symbol
-		(lib_id "Connector_Generic:Conn_01x01")
-		(at 77.47 55.88 180)
-		(unit 1)
-		(exclude_from_sim no)
-		(in_bom yes)
-		(on_board yes)
-		(dnp no)
-		(property "Reference" "J14"
-			(at 75.438 55.88 0)
-			(effects
-				(font
-					(size 1.27 1.27)
-				)
-				(justify left)
-			)
-		)
-		(property "Value" "Conn_01x01"
-			(at 74.93 54.6101 0)
-			(effects
-				(font
-					(size 1.27 1.27)
-				)
-				(justify left)
-				(hide yes)
-			)
-		)
-		(property "Footprint" "TestPoint:TestPoint_Pad_2.5x2.5mm"
-			(at 77.47 55.88 0)
-			(effects
-				(font
-					(size 1.27 1.27)
-				)
-				(hide yes)
-			)
-		)
-		(property "Datasheet" "~"
-			(at 77.47 55.88 0)
-			(effects
-				(font
-					(size 1.27 1.27)
-				)
-				(hide yes)
-			)
-		)
-		(property "Description" "Generic connector, single row, 01x01, script generated (kicad-library-utils/schlib/autogen/connector/)"
-			(at 77.47 55.88 0)
-			(effects
-				(font
-					(size 1.27 1.27)
-				)
-				(hide yes)
-			)
-		)
-		(pin "1"
-		)
-		(instances
-			(project "RemBreak"
-				(path "/e6d4ae5b-c9d7-4cbe-b288-c929fdf55a75/2d0cc746-3115-4ebf-adba-86e7fd6ac8bd"
-					(reference "J14")
-					(unit 1)
-				)

Commit message: changed size of the board and development of schematic
Parts:
- added D1: LED_ABGR, symbol Device:LED_ABGR
Connections:
- net 3V3: now also D1.1 (A)
- net Red: now reaches Q11.1 (C), Q12.3 (C), R27.1
Changed lines of the file:
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@@
+	(wire
+		(pts
+			(xy 147.32 153.67) (xy 147.32 157.48)
+		)
+		(stroke
+			(width 0)
+			(type default)
+		)
+	)
 	(wire
 		(pts
@@
 		)
 	)
+	(label "3V3"
+		(at 147.32 153.67 270)
+		(fields_autoplaced yes)
+		(effects
+			(font
+				(size 1.27 1.27)
+			)
+			(justify right bottom)
+		)
+	)
 	(label "5V"
 		(at 266.7 49.53 0)
@@
 			)
 			(justify left bottom)
+		)
+	)
+	(global_label "Red"
+		(shape input)
+		(at 109.22 68.58 180)
+		(fields_autoplaced yes)
+		(effects
+			(font
+				(size 1.27 1.27)
+			)
+			(justify right)
+		)
+		(property "Intersheetrefs" "${INTERSHEET_REFS}"
+			(at 102.7272 68.58 0)
+			(effects
+				(font
+					(size 1.27 1.27)
+				)
+				(justify right)
+				(hide yes)
+			)
 		)
 	)
@@
 					(unit 1)
 				)
+			)
+		)
+	)
+	(symbol
+		(lib_id "Device:LED_ABGR")
+		(at 147.32 162.56 90)
+		(unit 1)
+		(exclude_from_sim no)
+		(in_bom yes)
+		(on_board yes)
+		(dnp no)
+		(fields_autoplaced yes)
+		(property "Reference" "D1"
+			(at 156.21 161.2899 90)
+			(effects
+				(font
+					(size 1.27 1.27)
+				)
+				(justify right)
+			)
+		)
+		(property "Value" "LED_ABGR"
+			(at 156.21 163.8299 90)
+			(effects
+				(font
+					(size 1.27 1.27)
+				)
+				(justify right)
+			)
+		)
+		(property "Footprint" ""
+			(at 148.59 162.56 0)
+			(effects
+				(font
+					(size 1.27 1.27)
+				)
+				(hide yes)
+			)
+		)
+		(property "Datasheet" "~"
+			(at 148.59 162.56 0)
+			(effects
+				(font
+					(size 1.27 1.27)
+				)
+				(hide yes)
+			)
+		)
+		(property "Description" "RGB LED, anode/blue/green/red"
+			(at 147.32 162.56 0)
+			(effects
+				(font
+					(size 1.27 1.27)
+				)
+				(hide yes)
+			)
+		)
+		(pin "1"
+		)
+		(pin "3"
+		)
+		(pin "4"
+		)
+		(pin "2"
+		)
+		(instances
+			(project ""
+				(path "/e6d4ae5b-c9d7-4cbe-b288-c929fdf55a75/2d0cc746-3115-4ebf-adba-86e7fd6ac8bd"
+					(reference "D1")
+					(unit 1)
+				)

Commit message: added RGB LED connection - missing connections in schematics
Parts:
- removed D1: LED_ABGR, symbol Device:LED_ABGR
Connections:
- net RUNNIG: now reaches Q3.3 (C), Q9.1 (C), R10.1, U3.3 (CE), U4.3 (EN)
- net Red: no longer names the net of Q11.1 (C), Q12.3 (C), R27.1
Changed lines of the file:
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@@
+	)
+	(junction
+		(at 234.95 100.33)
+		(diameter 0)
+		(color 0 0 0 0)
 	)
 	(junction
@@
 	(wire
 		(pts
-			(xy 147.32 153.67) (xy 147.32 157.48)
+			(xy 234.95 100.33) (xy 273.05 100.33)
 		)
 		(stroke
@@
 		)
 	)
-	(label "3V3"
-		(at 147.32 153.67 270)
-		(fields_autoplaced yes)
-		(effects
-			(font
-				(size 1.27 1.27)
-			)
-			(justify right bottom)
-		)
-	)
 	(label "5V"
 		(at 266.7 49.53 0)
@@
 			)
 			(justify left bottom)
-		)
-	)
-	(global_label "Red"
-		(shape input)
-		(at 109.22 68.58 180)
-		(fields_autoplaced yes)
-		(effects
-			(font
-				(size 1.27 1.27)
-			)
-			(justify right)
-		)
-		(property "Intersheetrefs" "${INTERSHEET_REFS}"
-			(at 102.7272 68.58 0)
-			(effects
-				(font
-					(size 1.27 1.27)
-				)
-				(justify right)
-				(hide yes)
-			)
 		)
 	)
@@
 		(shape output)
 		(at 273.05 72.39 0)
+		(fields_autoplaced yes)
+		(effects
+			(font
+				(size 1.27 1.27)
+			)
+			(justify left)
+		)
+	)
+	(hierarchical_label "RUNNIG"
+		(shape input)
+		(at 273.05 100.33 0)
 		(fields_autoplaced yes)
 		(effects
@@
 					(unit 1)
 				)
-			)
-		)
-	)
-	(symbol
-		(lib_id "Device:LED_ABGR")
-		(at 147.32 162.56 90)
-		(unit 1)
-		(exclude_from_sim no)
-		(in_bom yes)
-		(on_board yes)
-		(dnp no)
-		(fields_autoplaced yes)
-		(property "Reference" "D1"
-			(at 156.21 161.2899 90)
-			(effects
-				(font
-					(size 1.27 1.27)
-				)
-				(justify right)
-			)
-		)
-		(property "Value" "LED_ABGR"
-			(at 156.21 163.8299 90)
-			(effects
-				(font
-					(size 1.27 1.27)
-				)
-				(justify right)
-			)
-		)
-		(property "Footprint" ""
-			(at 148.59 162.56 0)
-			(effects
-				(font
-					(size 1.27 1.27)
-				)
-				(hide yes)
-			)
-		)
-		(property "Datasheet" "~"
-			(at 148.59 162.56 0)
-			(effects
-				(font
-					(size 1.27 1.27)
-				)
-				(hide yes)
-			)
-		)
-		(property "Description" "RGB LED, anode/blue/green/red"
-			(at 147.32 162.56 0)
-			(effects
-				(font
-					(size 1.27 1.27)
-				)
-				(hide yes)
-			)
-		)
-		(pin "1"
-		)
-		(pin "3"
-		)
-		(pin "4"
-		)
-		(pin "2"
-		)
-		(instances
-			(project ""
-				(path "/e6d4ae5b-c9d7-4cbe-b288-c929fdf55a75/2d0cc746-3115-4ebf-adba-86e7fd6ac8bd"
-					(reference "D1")
-					(unit 1)
-				)
