File: hw/RFController/RFController.kicad_sch (KiCad schematic)
At the start: 19 parts, among them J1 Conn_01x07, J2 Conn_01x01, SW1 SW_Push, U1 ADC128D818, Y1 Crystal

Commit message: rf controller added crystal 3d model
Changed lines of the file:
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@@
 (kicad_sch
-	(version 20231120)
+	(version 20241004)
 	(generator "eeschema")
-	(generator_version "8.0")
+	(generator_version "8.99")
 	(paper "A4")
 	(symbol
@@
 		)
 	)
+	(embedded_fonts no)
 )
