File: hw/prototyping/breakoutpcbs/breakoutpcbs.kicad_pcb (KiCad board)
At the start: 2 copper layers, 143.8 x 99.6 mm, 108 parts, among them IC1 LTC2943IDD#TRPBF, J1 Conn_01x05, J10 Conn_01x03_MountingPin, J11 Conn_01x07, J12 Conn_01x07, J13 Conn_01x06, J14 Conn_01x02, J15 Conn_01x04, J16 Screw_Terminal_01x04, J17 Conn_01x05, J18 Screw_Terminal_01x04, J19 Conn_01x02, J2 Conn_01x05, J3 Conn_01x07, J4 Conn_01x02, J5 Conn_01x03, J6 Conn_01x05, J7 Conn_01x02, J8 Conn_01x02, J9 Screw_Terminal_01x02, Q1 BC337, Q10 BC337, Q11 BC847, Q2 BC847, Q3 BC847, Q4 BC337, Q5 BC337, Q6 SiS415DNT, Q7 BC847, Q8 BC337, Q9 BC847, U1 INA219BxDCN, U2 BD48ExxG, U3 L7805, U4 XC6220B331MR, U5 MAX40200AUK, U6 BD48ExxG, U7 BD48ExxG, U8 MAX40200AUK, U9 MAX40200AUK

Commit message: updated schematics
Parts:
- R11: value 50k -> 91k
- R12: value 100k -> 67k
- R31: value 10k -> 0R
- R40: value 4k7 -> 2k7
- R41: value 10k -> 4k7
- R47, R6, R7: value 4k2 -> 0R
Changed lines of the file:
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@@
 		(sheetname "/power_switch_bbB/")
 		(sheetfile "power_switch_bbB.kicad_sch")
-		(attr smd)
+		(attr smd dnp)
 		(fp_line
 			(start -0.227064 -0.735)
@@
 			)
 		)
-		(property "Value" "50k"
+		(property "Value" "91k"
 			(at 0 1.65 90)
 			(layer "F.Fab")
@@
 			)
 		)
-		(property "Value" "10k"
+		(property "Value" "4k7"
 			(at 0 1.65 90)
 			(layer "F.Fab")
@@
 			)
 		)
-		(property "Value" "4k7"
+		(property "Value" "2k7"
 			(at 0 1.65 0)
 			(layer "F.Fab")
@@
 		(sheetname "/power_switch_bbB/")
 		(sheetfile "power_switch_bbB.kicad_sch")
-		(attr smd dnp)
+		(attr smd)
 		(fp_line
 			(start -0.227064 -0.735)
@@
 		(sheetname "/power_switch_bbA/")
 		(sheetfile "power_switch_bbA.kicad_sch")
-		(attr smd dnp)
+		(attr smd)
 		(fp_line
 			(start -0.227064 0.735)
@@
 		(sheetname "/power_switch_bbA/")
 		(sheetfile "power_switch_bbA.kicad_sch")
-		(attr smd)
+		(attr smd dnp)
 		(fp_line
 			(start -0.727064 -0.91)
@@
 			)
 		)
-		(property "Value" "10k"
+		(property "Value" "0R"
 			(at 0 1.65 0)
 			(layer "F.Fab")
@@
 			)
 		)
-		(property "Value" "100k"
+		(property "Value" "67k"
 			(at 0 1.65 90)
 			(layer "F.Fab")
@@
 		(sheetname "/power_switch_bbA/")
 		(sheetfile "power_switch_bbA.kicad_sch")
-		(attr smd dnp)
+		(attr smd)
 		(fp_line
 			(start -0.227064 -0.735)
@@
 			)
 		)
-		(property "Value" "4k2"
+		(property "Value" "0R"
 			(at 0 1.65 0)
 			(layer "F.Fab")
@@
 		(sheetname "/power_switch_bbA/")
 		(sheetfile "power_switch_bbA.kicad_sch")
-		(attr smd dnp)
+		(attr smd)
 		(fp_line
 			(start -0.227064 -0.735)
@@
 			)
 		)
-		(property "Value" "4k2"
+		(property "Value" "0R"
 			(at 0 1.65 0)
 			(layer "F.Fab")
@@
 			)
 		)
-		(property "Value" "4k2"
+		(property "Value" "0R"
 			(at 0 1.65 0)
 			(layer "F.Fab")
