File: hw/prototyping/breakoutpcbs/power_manager_bb.kicad_sch (KiCad schematic)
At the start: 8 parts, among them IC1 LTC2943IDD#TRPBF, J1 Conn_01x05, J2 Conn_01x05, U1 INA219BxDCN

Commit message: updated kicad version and updated todo list with different found issues
Parts:
- R3: value 001R -> 002R
Changed lines of the file:
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@@
 (kicad_sch
-	(version 20241209)
+	(version 20250114)
 	(generator "eeschema")
 	(generator_version "9.0")
@@
 			)
 		)
-		(property "Value" "001R"
+		(property "Value" "002R"
 			(at 149.86 78.74 90)
 			(effects
