File: hw/prototyping/breakoutpcbs/power_switch_bbA.kicad_sch (KiCad schematic)
At the start: 27 parts, among them J5 Conn_01x03, J7 Conn_01x02, J8 Conn_01x02, Q3 BC847, Q4 BC337, Q5 BC337, Q6 SiS415DNT, Q7 BC847, U6 BD48ExxG

Commit message: refactoring of the current boards and two added to test the whole circuit
Parts:
- added R29: 4k2, Resistor_SMD:R_0805_2012Metric_Pad1.20x1.40mm_HandSolder, symbol Device:R
- added R30: 10k, Resistor_SMD:R_0805_2012Metric_Pad1.20x1.40mm_HandSolder, symbol Device:R
- added R33: 0R, Resistor_SMD:R_1206_3216Metric, symbol Device:R
- R17, R21, R23: now not fitted
- R20: value 4k2 -> 0R
Connections:
- net at R15.1, R16.2, R17.1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: now also R29.1, R33.2
- net at Q3.1 (B), Q4.2 (B), R14.2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: now also R33.1
- net at Q6.4 (G), R19.2, R23.2: now also R30.2
- net at Q5.2 (B), Q7.1 (B), R17.2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: now also R30.1
- net at Q5.1 (C), Q7.3 (C), R23.1: now also R29.2
Other:
- moved on the sheet: Q5, Q7, R26, R27

Commit message: updated schematics
Parts:
- R11: value 50k -> 91k
- R12: value 100k -> 67k
- R17, R21, R23: now fitted
- R33: now not fitted
Connections:
- net RUNNING: now reaches Q5.1 (C), Q7.3 (C), R23.1, R29.2
Changed lines of the file:
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@@
+		)
+	)
+	(label "RUNNING"
+		(at 193.04 57.15 0)
+		(effects
+			(font
+				(size 1.27 1.27)
+			)
+			(justify left bottom)
 		)
 	)
@@
 		(in_bom yes)
 		(on_board yes)
-		(dnp no)
+		(dnp yes)
 		(fields_autoplaced yes)
 		(property "Reference" "R33"
@@
 		(in_bom yes)
 		(on_board yes)
-		(dnp yes)
+		(dnp no)
 		(fields_autoplaced yes)
 		(property "Reference" "R21"
@@
 			)
 		)
-		(property "Value" "50k"
+		(property "Value" "91k"
 			(at 72.644 77.47 90)
 			(effects
@@
 		(in_bom yes)
 		(on_board yes)
-		(dnp yes)
+		(dnp no)
 		(fields_autoplaced yes)
 		(property "Reference" "R17"
@@
 			)
 		)
-		(property "Value" "100k"
+		(property "Value" "67k"
 			(at 72.644 106.68 90)
 			(effects
@@
 		(in_bom yes)
 		(on_board yes)
-		(dnp yes)
+		(dnp no)
 		(property "Reference" "R23"
 			(at 169.926 41.148 0)
