File: hw/breakoutpcbs/power_switch_bbB.kicad_sch (KiCad schematic)
At the start: 27 parts, among them J3 Conn_01x07, J4 Conn_01x02, Q1 BC337, Q2 BC847, U2 BD48ExxG, U3 L7805, U4 XC6220B331MR, U5 MAX40200AUK, U7 BD48ExxG

Commit message: new todos, the charging signal removed, plugged signal used instead
Other:
- note added: "TODO: add shottky diode - maybe add bypass resistor don't know if the DC/DC will have lower parallel resistance"
- note added: "TODO: signal "plugged" Resistor ~18k in parallel with Q1 connect to MCU as charging pin"
Changed lines of the file:
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@@
 		(title "Power Switch Breakout Board")
+	)
+	(text "TODO: signal \"plugged\" \nResistor ~18k in parallel with Q1\nconnect to MCU as charging pin"
+		(exclude_from_sim no)
+		(at 137.16 108.966 0)
+		(effects
+			(font
+				(size 1.27 1.27)
+			)
+		)
+	)
+	(text "TODO: add shottky diode\n- maybe add bypass resistor\ndon't know if the DC/DC will have lower\nparallel resistance"
+		(exclude_from_sim no)
+		(at 90.17 24.638 0)
+		(effects
+			(font
+				(size 1.27 1.27)
+			)
+		)
 	)
 	(text "adjust the threshold\nto 4V"

Commit message: updated breakoutboards components attributes
Other:
- note added: "disconnect"
Changed lines of the file:
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@@
+		)
+	)
+	(text "disconnect"
+		(exclude_from_sim no)
+		(at 155.702 126.238 0)
+		(effects
+			(font
+				(size 1.27 1.27)
+			)
 		)
 	)
@@
 	(wire
 		(pts
+			(xy 107.95 74.93) (xy 107.95 99.06)
+		)
+		(stroke
+			(width 0)
+			(type default)
+		)
+	)
+	(wire
+		(pts
 			(xy 67.31 87.63) (xy 67.31 119.38)
 		)
@@
 		(pts
 			(xy 86.36 60.96) (xy 86.36 62.23)
-		)
-		(stroke
-			(width 0)
-			(type default)
-		)
-	)
-	(wire
-		(pts
-			(xy 107.95 74.93) (xy 107.95 99.06)
 		)
 		(stroke
@@
 		)
 	)
+	(rule_area
+		(polyline
+			(pts
+				(xy 62.23 93.98) (xy 62.23 151.13) (xy 149.86 151.13) (xy 149.86 93.98)
+			)
+			(stroke
+				(width 0)
+				(type dash)
+			)
+			(fill
+				(type none)
+			)
+		)
+	)
